File: proudova_pojistka/untitled.kicad_sch (KiCad schematic)
At the start: 2 parts, among them U1 L78L05_SOT89

Commit message: Napájení
Parts:
- added C10, C2, C3, C4, C5, C7: 100n, Capacitor_THT:C_Disc_D5.0mm_W2.5mm_P5.00mm, symbol Device:C_Small
- added C8, C9: 220u/25, Capacitor_THT:CP_Radial_D8.0mm_P3.50mm, symbol Device:C_Polarized_Small
- added D1, D2: 1N4148, Diode_THT:D_DO-35_SOD27_P7.62mm_Horizontal, symbol Diode:1N4148
- added J1: Napájení +12V, TerminalBlock_Phoenix:TerminalBlock_Phoenix_MKDS-1,5-2-5.08_1x02_P5.08mm_Horizontal, symbol Connector:Screw_Terminal_01x02
- added R1: 1k, Resistor_THT:R_Axial_DIN0918_L18.0mm_D9.0mm_P22.86mm_Horizontal, symbol Device:R_Small
- added U2: NE555P, Package_DIP:DIP-8_W7.62mm, symbol Timer:NE555P
- C1: value C_Polarized_Small -> 220u/25; footprint (none) -> Capacitor_THT:CP_Radial_D8.0mm_P3.50mm
Connections:
- net +5V: now reaches U1.1 (OUT)
- net +5V: now also C3.1
- net GND: now reaches U1.2 (GND)
- net GND: now also C1.2, C10.2, C2.2, C3.2, C4.2, C5.2, C7.2, C9.1, D2.1 (K), J1.1 (Pin_1), U2.1 (GND)
- net +12V: now reaches U1.3 (IN)
- net +12V: now also C1.1, C2.1, C4.1, J1.2 (Pin_2)
- new net: C10.1, R1.2, U2.2 (TR), U2.6 (THR)
- new net: C8.1, R1.1, U2.3 (Q)
- new net: C7.1, U2.5 (CV)
- new net: C8.2, D1.1 (K), D2.2 (A)
- new net -10V: C9.2, D1.2 (A)
- new net -12V: C5.1, U2.4 (R)
- no-connect marks 0 -> 1
Other:
- moved on the sheet: C1, U1

Commit message: Schéma + Footprinty
Connections:
- net -12V is gone; now on net +12V: C5.1, U2.4 (R)
- net +12V: now also U2.8 (VCC)
Other:
- moved on the sheet: C5
